Commit message: updated planar lidar and slamtoolbox

File: husky_panda_description/husky_panda_model/panda_mounted_husky/husky_robot_description/husky.urdf.xacro (robot description, xacro)
@@ -62,16 +62,16 @@
           </geometry>
         </visual>
-        <visual name="front_bumper_visual">
+        <!-- <visual name="front_bumper_visual">
           <origin xyz="0.48 0 0.091" rpy="0 0 0"/>
           <geometry>
             <mesh filename="${husky_mesh_prefix}/bumper.dae"/>
           </geometry>
-        </visual>
-        <visual name="rear_bumper_visual">
+        </visual> -->
+        <!-- <visual name="rear_bumper_visual">
           <origin xyz="-0.48 0 0.091" rpy="0 0 3.14159"/>
           <geometry>
             <mesh filename="${husky_mesh_prefix}/bumper.dae"/>
           </geometry>
-        </visual>
+        </visual> -->
         <visual name="top_chassis_visual">
           <origin xyz="0 0 0" rpy="0 0 0"/>
@@ -105,4 +105,6 @@
         </visual>
         <visual name="planar_lidar_visual">
+          <!-- <origin xyz="0.474 0 0.127" rpy="0 0 0"/> -->
+            <!-- was: 0.474 0 0.127 0 0 0 -->
           <origin xyz="0.474 0 0.127" rpy="0 0 0"/>
           <geometry>
@@ -371,4 +373,5 @@
         <sensor name="planar_laser" type="gpu_ray">
         <topic>planar_laser</topic>
+          <!-- <pose>0.474 0 0.127 0 0 0</pose> -->
           <pose>0.474 0 0.127 0 0 0</pose>
           <update_rate>10</update_rate>
@@ -383,5 +386,5 @@
             </scan>
             <range>
-              <min>0.20</min>
+              <min>0.60</min>
               <max>25.0</max>
               <resolution>0.01</resolution>
@@ -560,4 +563,5 @@
         <parent link="base_link"/>
         <child link="planar_lidar_link"/>
+        <!-- <origin xyz="0.474 0 0.127" rpy="0 0 0"/> -->
         <origin xyz="0.474 0 0.127" rpy="0 0 0"/>
       </joint>

File: husky_panda_description/husky_panda_model/panda_mounted_husky/panda_mount_husky.urdf (robot description, URDF)
Before this commit: robot panda_mounted_husky, 25 links, 24 joints
Links:
- link base_link: geometry collision box size=0.2 0.25 0.225; collision box size=0.500 0.385 0.155

Commit message: integrated lio sam

File: husky_panda_description/husky_panda_model/panda_mounted_husky/husky_robot_description/husky.urdf.xacro (robot description, xacro)
@@ -270,4 +270,39 @@
         </visual>
       </link>
+      <!-- camera_pan_tilt on the gimbal -->
+    <gazebo reference="tilt_gimbal_link">
+      <sensor name="camera_pan_tilt" type="rgbd_camera">
+        <topic>camera_pan_tilt</topic>
+        <pose>0 0 0.03 0 0 0</pose>
+        <update_rate>30</update_rate>
+        <camera name="camera_pan_tilt">
+          <horizontal_fov>1.5184</horizontal_fov>
+          <lens>
+            <intrinsics>
+              <fx>337.22195</fx>
+              <fy>337.22195</fy>
+              <cx>320.5</cx>
+              <cy>240.5</cy>
+              <s>0</s>
+            </intrinsics>
+          </lens>
+          <distortion>
+            <k1>0.0</k1><k2>0.0</k2><k3>0.0</k3>
+            <p1>0.0</p1><p2>0.0</p2>
+            <center>0.5 0.5</center>
+          </distortion>
+          <image>
+            <width>640</width>
+            <height>480</height>
+            <format>R8G8B8</format>
+          </image>
+          <clip><near>0.01</near><far>300</far></clip>
+          <depth_camera><clip><near>0.1</near><far>10</far></clip></depth_camera>
+          <noise>
+            <type>gaussian</type><mean>0</mean><stddev>0.007</stddev>
+          </noise>
+        </camera>
+      </sensor>
+    </gazebo>
       <!-- planar_lidar_link -->
       <link name="planar_lidar_link"/>
@@ -338,5 +373,5 @@
             </distortion>
             <image>
-              <width>320</width><height>240</height><format>R8G8B8</format>
+              <width>640</width><height>480</height><format>R8G8B8</format>
             </image>
             <clip><near>0.01</near><far>300</far></clip>
@@ -363,5 +398,5 @@
             </distortion>
             <image>
-              <width>320</width><height>240</height><format>R8G8B8</format>
+              <width>640</width><height>480</height><format>R8G8B8</format>
             </image>
             <clip><near>0.01</near><far>300</far></clip>

File: husky_panda_description/husky_panda_model/panda_mounted_husky/panda_model_description/panda.urdf.xacro (robot description, xacro)
@@ -100,18 +100,27 @@
   </link>
   <!-- SDF frame as massless link -->
-  <link name="wrist_mount"/>
+  <link name="gripper_mount"/>
   <!-- Camera body (small mass to keep physics stable) -->
-  <link name="wrist_cam_link">
+  <link name="gripper_cam_link">
     <inertial>
       <mass value="0.08"/>
       <origin xyz="0 0 0" rpy="0 0 0"/>
-      <inertia ixx="0.0001" iyy="0.0001" izz="0.0001" ixy="0" ixz="0" iyz="0"/>
-    </inertial>
-    <visual name="wrist_cam_debug">
-      <geometry><box size="0.06 0.02 0.02"/></geometry>
+       <inertia ixx="1.8e-4" iyy="5.0e-5" izz="1.8e-4" ixy="0" ixz="0" iyz="0"/>
+    </inertial>
+     <visual name="realsense_d415_vis">
+      <origin xyz="0 -0.02 0" rpy="1.57079632679 0 1.57079632679"/>
+      <geometry>
+        <mesh filename="${panda_mesh_prefix}/d415.stl" scale="0.001 0.001 0.001"/>
+      </geometry>
     </visual>
-  </link>
+    <collision name="realsense_d415_col">
+      <origin xyz="-0.0125 -0.02 0" rpy="0 0 0"/>
+      <geometry>
+        <box size="0.02005 0.099 0.023"/>
+      </geometry>
+    </collision>
+     </link>
   <!-- REP 103 optical frame -->
-  <link name="wrist_cam_optical_frame"/>
+  <link name="gripper_cam_optical_frame"/>
   <!-- Fingers -->
   <link name="panda_leftfinger">
@@ -198,15 +207,15 @@
   </joint>
   <!-- fixed frames -->
-  <joint name="panda_wrist_mount" type="fixed">
-    <parent link="panda_link7"/><child link="wrist_mount"/>
+  <joint name="panda_gripper_mount" type="fixed">
+    <parent link="panda_link7"/><child link="gripper_mount"/>
     <origin xyz="0 0 0.107" rpy="0 0 -0.7853981633974483"/>
   </joint>
-  <joint name="wrist_cam_mount" type="fixed">
-    <parent link="wrist_mount"/><child link="wrist_cam_link"/>
-    <!-- SDF had +5 cm forward from wrist_mount -->
+  <joint name="gripper_cam_mount" type="fixed">
+    <parent link="gripper_mount"/><child link="gripper_cam_link"/>
+    <!-- SDF had +5 cm forward from gripper_mount -->
     <origin xyz="0 0 0.05" rpy="0 0 0"/>
   </joint>
-  <joint name="wrist_cam_optical_joint" type="fixed">
-    <parent link="wrist_cam_link"/><child link="wrist_cam_optical_frame"/>
+  <joint name="gripper_cam_optical_joint" type="fixed">
+    <parent link="gripper_cam_link"/><child link="gripper_cam_optical_frame"/>
     <!-- Z forward, X right, Y down -->
     <origin xyz="0 0 0" rpy="-1.57079632679 0 -1.57079632679"/>
@@ -245,14 +254,14 @@
     <joint name="panda_joint6"><command_interface name="position"/><state_interface name="position"/><state_interface name="velocity"/><state_interface name="effort"/></joint>
     <joint name="panda_joint7"><command_interface name="position"/><state_interface name="position"/><state_interface name="velocity"/><state_interface name="effort"/></joint>
-    <!-- wrist fingers -->
+    <!-- gripper fingers -->
     <joint name="panda_finger_joint1"><command_interface name="position"/><state_interface name="position"/><state_interface name="velocity"/></joint>
     <joint name="panda_finger_joint2"><command_interface name="position"/><state_interface name="position"/><state_interface name="velocity"/></joint>
   </ros2_control>
   <!-- ================== Gazebo: load ros2_control, friction, and sensor ================== -->
-  <!-- <gazebo>
+  <gazebo>
     <plugin filename="libgz_ros2_control-system.so" name="gz_ros2_control::GazeboSimROS2ControlPlugin">
-      <parameters>/config/controllers.yaml</parameters>
-    </plugin>
-  </gazebo> -->
+      <parameters>/home/rebellion/mobile_robotics/gz_start/robot_models/panda_arm_model/colcon_ws/src/husky_panda_description/config/controller.yaml</parameters>
+    </plugin>
+  </gazebo>
   <gazebo reference="panda_link0"><gravity>false</gravity></gazebo>
   <gazebo>
@@ -364,11 +373,11 @@
   <gazebo reference="panda_rightfinger"><mu1>1.13</mu1><mu2>1.13</mu2></gazebo>
   <!-- Embed the RGB-D sensor (GZ Sim understands SDF inside <gazebo> in URDF) -->
-  <gazebo reference="wrist_cam_link">
-    <sensor name="wrist_rgbd" type="rgbd_camera">
+  <gazebo reference="gripper_cam_link">
+    <sensor name="gripper_rgbd" type="rgbd_camera">
       <pose>0.015 0 0 0 -1.57079632679 0</pose>
       <update_rate>30</update_rate>
       <always_on>true</always_on>
       <visualize>true</visualize>
-      <topic>/panda/wrist/rgbd</topic>
+      <topic>/panda/gripper/rgbd</topic>
       <camera>
         <horizontal_fov>1.0471975512</horizontal_fov>

File: husky_panda_description/husky_panda_model/panda_mounted_husky/panda_mount_husky.urdf (robot description, URDF)
Before this commit: robot panda_mounted_husky, 25 links, 24 joints
Links:
- removed link wrist_cam_link
- removed link wrist_cam_optical_frame
- removed link wrist_mount
- added link gripper_cam_link, mass 0.08; visual box size=0.06 0.02 0.02
- added link gripper_cam_optical_frame
- added link gripper_mount
Joints:
- removed joint panda_wrist_mount
- removed joint wrist_cam_mount
- removed joint wrist_cam_optical_joint
- added joint gripper_cam_mount: type fixed, parent gripper_mount, child gripper_cam_link, origin xyz=0 0 0.05 rpy=0 0 0
- added joint gripper_cam_optical_joint: type fixed, parent gripper_cam_link, child gripper_cam_optical_frame, origin xyz=0 0 0 rpy=-1.57079632679 0 -1.57079632679
- added joint panda_gripper_mount: type fixed, parent panda_link7, child gripper_mount, origin xyz=0 0 0.107 rpy=0 0 -0.7853981633974483
