Commit message: Recommit current state (exclude large zip)

File: husky_panda_description/husky_panda_model/panda_mounted_husky/panda_mounted_husky.urdf.xacro (robot description, xacro)
@@ -1,20 +1,900 @@
 <?xml version="1.0"?>
-<robot name="panda_mounted_husky" xmlns:xacro="http://www.ros.org/wiki/xacro">
-  <!-- Tune the mount offset as you like -->
-  <!-- <xacro:arg name="mount_xyz" default="0 0 0.2325"/>
-  <xacro:arg name="mount_rpy" default="0 0 0"/> -->
-  <!-- Include macros (use RELATIVE paths so xacro doesn't need find-pkg-share) -->
-  <xacro:include filename="husky_robot_description/husky.urdf.xacro"/>
-  <xacro:include filename="panda_model_description/panda.urdf.xacro"/>
-  <!-- Instantiate Husky and Panda for RViz.
-       Keep Panda joint names EXACTLY as 'panda_joint{1..7}', etc.
-       (Your sliders & husky_panda_bridge depend on those names.) -->
-  <xacro:husky/>        <!-- leaves base link as 'base_link' -->
-  <xacro:panda/>        <!-- keeps joints 'panda_joint1'.. etc. -->
-  <!-- ONE rigid joint between them so URDF is a single tree -->
+<robot xmlns:xacro="http://www.ros.org/wiki/xacro" name="panda_mounted_husky">
+    <!-- <xacro:property name="mesh_root"
+         value="package://husky_panda_description/husky_panda_model/panda_mounted_husky/meshes"/>   -->
+    <!-- =========================
+       HUSKY BASE
+       ========================= -->
+      <!-- =========================
+          LINKS
+          ========================= -->
+      <!-- base_link -->
+      <link name="base_link">
+        <inertial>
+          <origin xyz="-0.000543 -0.084945 0.062329" rpy="0 0 0"/>
+          <mass value="46.064"/>
+          <inertia
+            ixx="0.615397" ixy="-0.0240585" ixz="-0.120749"
+            iyy="1.75388"  iyz="-0.0028322" izz="2.03641"/>
+        </inertial>
+        <!-- <joint name="base_footprint_joint" type="fixed">
+            <parent link="base_link"/>
+            <child link="base_footprint"/>
+            <origin xyz="0 0 0" rpy="0 0 0"/>
+        </joint>
+        <link name="base_footprint">
+        </link> -->
+        <!-- Collisions -->
+        <collision name="base_link_collision">
+          <origin xyz="0 0 0.12" rpy="0 0 0"/>
+          <geometry>
+            <box size="0.9874 0.5709 0.05"/>
+          </geometry>
+        </collision>
+        <collision name="base_link_collision_bottom">
+          <origin xyz="0 0 0.046" rpy="0 0 0"/>
+          <geometry>
+            <box size="0.80 0.5709 0.095"/>
+          </geometry>
+        </collision>
+        <collision name="base_link_collision_1">
+          <origin xyz="0 0 0.185625" rpy="0 0 0"/>
+          <geometry>
+            <box size="0.78992 0.5709 0.12375"/>
+          </geometry>
+        </collision>
+        <collision name="sensor_tower_collision">
+          <origin xyz="0.374 0 0.215" rpy="0 0 0"/>
+          <geometry>
+            <box size="0.2 0.25 0.225"/>
+          </geometry>
+        </collision>
+        <collision name="landing_pad_collision">
+          <origin xyz="0.0 0 0.155" rpy="0 0 0"/>
+          <geometry>
+            <box size="0.500 0.385 0.155"/>
+          </geometry>
+        </collision>
+        <!-- Visuals -->
+        <visual name="base_link_visual">
+          <origin xyz="0 0 0" rpy="0 0 0"/>
+          <geometry>
+            <mesh filename="package://husky_panda_description/husky_panda_model/panda_mounted_husky/meshes/base_link.dae" scale="1 1 1"/>
+          </geometry>
+        </visual>
+        <!-- <visual name="front_bumper_visual">
+          <origin xyz="0.48 0 0.091" rpy="0 0 0"/>
+          <geometry>
+            <mesh filename="package://husky_panda_description/husky_panda_model/panda_mounted_husky/meshes/bumper.dae"/>
+          </geometry>
+        </visual> -->
+        <!-- <visual name="rear_bumper_visual">
+          <origin xyz="-0.48 0 0.091" rpy="0 0 3.14159"/>
+          <geometry>
+            <mesh filename="package://husky_panda_description/husky_panda_model/panda_mounted_husky/meshes/bumper.dae"/>
+          </geometry>
+        </visual> -->
+        <visual name="top_chassis_visual">
+          <origin xyz="0 0 0" rpy="0 0 0"/>
+          <geometry>
+            <mesh filename="package://husky_panda_description/husky_panda_model/panda_mounted_husky/meshes/top_chassis.dae"/>
+          </geometry>
+        </visual>
+        <visual name="velodyne_base_visual_1">
+          <origin xyz="0.424 0 0.327" rpy="0 0 0"/>
+          <geometry>
+            <mesh filename="package://husky_panda_description/husky_panda_model/panda_mounted_husky/meshes/VLP16_base_1.dae"/>
+          </geometry>
+        </visual>
+        <visual name="velodyne_base_visual_2">
+          <origin xyz="0.424 0 0.327" rpy="0 0 0"/>
+          <geometry>
+            <mesh filename="package://husky_panda_description/husky_panda_model/panda_mounted_husky/meshes/VLP16_base_2.dae"/>
+          </geometry>
+        </visual>
+        <visual name="velodyne_scan_visual">
+          <origin xyz="0.424 0 0.327" rpy="0 0 0"/>
+          <geometry>
+            <mesh filename="package://husky_panda_description/husky_panda_model/panda_mounted_husky/meshes/VLP16_scan.dae"/>
+          </geometry>
+        </visual>
+        <visual name="user_rail_visual">
+          <origin xyz="0.272 0 0.245" rpy="0 0 0"/>
+          <geometry>
+            <mesh filename="package://husky_panda_description/husky_panda_model/panda_mounted_husky/meshes/user_rail.dae"/>
+          </geometry>
+        </visual>
+        <visual name="planar_lidar_visual">
+          <!-- <origin xyz="0.474 0 0.127" rpy="0 0 0"/> -->
+            <!-- was: 0.474 0 0.127 0 0 0 -->
+          <origin xyz="0.474 0 0.127" rpy="0 0 0"/>
+          <geometry>
+            <cylinder radius="0.045" length="0.05"/>
+          </geometry>
+        </visual>
+        <visual name="sensor_tower_visual">
+          <origin xyz="0.374 0 0.215" rpy="0 0 0"/>
+          <geometry>
+            <box size="0.2 0.25 0.225"/>
+          </geometry>
+        </visual>
+        <visual name="landing_pad_visual">
+          <origin xyz="0.0 0 0.155" rpy="0 0 0"/>
+          <geometry>
+            <box size="0.500 0.385 0.155"/>
+          </geometry>
+        </visual>
+        <visual name="base_realsense_down_visual">
+          <origin xyz="0.478 0 0.260" rpy="0 -0.035 0"/>
+          <geometry>
+            <mesh filename="package://husky_panda_description/husky_panda_model/panda_mounted_husky/meshes/realsense.dae"/>
+          </geometry>
+        </visual>
+        <visual name="base_realsense_front_visual">
+          <origin xyz="0.478 0 0.285" rpy="0 0 0"/>
+          <geometry>
+            <mesh filename="package://husky_panda_description/husky_panda_model/panda_mounted_husky/meshes/realsense.dae"/>
+          </geometry>
+        </visual>
+      </link>
+      <!-- front_left_wheel_link -->
+      <link name="front_left_wheel_link">
+        <inertial>
+          <origin xyz="0 0 0"/>
+          <mass value="2.637"/>
+          <inertia ixx="0.02467" iyy="0.04411" izz="0.02467" ixy="0" ixz="0" iyz="0"/>
+        </inertial>
+        <collision>
+          <origin xyz="0 0 0" rpy="1.5707963267948966 0 0"/>
+          <geometry>
+            <cylinder radius="0.1651" length="0.1143"/>
+          </geometry>
+        </collision>
+        <visual>
+          <geometry>
+            <mesh filename="package://husky_panda_description/husky_panda_model/panda_mounted_husky/meshes/wheel.dae"/>
+          </geometry>
+        </visual>
+      </link>
+      <!-- front_right_wheel_link -->
+      <link name="front_right_wheel_link">
+        <inertial>
+          <origin xyz="0 0 0"/>
+          <mass value="2.637"/>
+          <inertia ixx="0.02467" iyy="0.04411" izz="0.02467" ixy="0" ixz="0" iyz="0"/>
+        </inertial>
+        <collision>
+          <origin xyz="0 0 0" rpy="1.5707963267948966 0 0"/>
+          <geometry>
+            <cylinder radius="0.1651" length="0.1143"/>
+          </geometry>
+        </collision>
+        <visual>
+          <geometry>
+            <mesh filename="package://husky_panda_description/husky_panda_model/panda_mounted_husky/meshes/wheel.dae"/>
+          </geometry>
+        </visual>
+      </link>
+      <!-- rear_left_wheel_link -->
+      <link name="rear_left_wheel_link">
+        <inertial>
+          <origin xyz="0 0 0"/>
+          <mass value="2.637"/>
+          <inertia ixx="0.02467" iyy="0.04411" izz="0.02467" ixy="0" ixz="0" iyz="0"/>
+        </inertial>
+        <collision>
+          <origin xyz="0 0 0" rpy="1.5707963267948966 0 0"/>
+          <geometry>
+            <cylinder radius="0.1651" length="0.1143"/>
+          </geometry>
+        </collision>
+        <visual>
+          <geometry>
+            <mesh filename="package://husky_panda_description/husky_panda_model/panda_mounted_husky/meshes/wheel.dae"/>
+          </geometry>
+        </visual>
+      </link>
+      <!-- rear_right_wheel_link -->
+      <link name="rear_right_wheel_link">
+        <inertial>
+          <origin xyz="0 0 0"/>
+          <mass value="2.637"/>
+          <inertia ixx="0.02467" iyy="0.04411" izz="0.02467" ixy="0" ixz="0" iyz="0"/>
+        </inertial>
+        <collision>
+          <origin xyz="0 0 0" rpy="1.5707963267948966 0 0"/>
+          <geometry>
+            <cylinder radius="0.1651" length="0.1143"/>
+          </geometry>
+        </collision>
+        <visual>
+          <geometry>
+            <mesh filename="package://husky_panda_description/husky_panda_model/panda_mounted_husky/meshes/wheel.dae"/>
+          </geometry>
+        </visual>
+      </link>
+      <!-- pan_gimbal_link -->
+      <link name="pan_gimbal_link">
+        <inertial>
+          <origin xyz="0 0 0"/>
+          <mass value="0.1"/>
+          <inertia ixx="0.000016875" iyy="1e-8" izz="0.000016875" ixy="0" ixz="0" iyz="0"/>
+        </inertial>
+        <collision>
+          <geometry>
+            <cylinder radius="0.014" length="0.045"/>
+          </geometry>
+        </collision>
+        <visual>
+          <geometry>
+            <cylinder radius="0.014" length="0.045"/>
+          </geometry>
+        </visual>
+      </link>
+      <!-- tilt_gimbal_link -->
+      <link name="tilt_gimbal_link">
+        <inertial>
+          <origin xyz="0 0 0" rpy="1.570796 0 0"/>
+          <mass value="0.1"/>
+          <inertia ixx="0.000016875" iyy="1e-8" izz="0.000016875" ixy="0" ixz="0" iyz="0"/>
+        </inertial>
+        <collision>
+          <origin rpy="1.570796 0 0"/>
+          <geometry>
+            <cylinder radius="0.014" length="0.045"/>
+          </geometry>
+        </collision>
+        <visual>
+          <origin rpy="1.570796 0 0"/>
+          <geometry>
+            <cylinder radius="0.014" length="0.045"/>
+          </geometry>
+        </visual>
+        <!-- Extra visuals on tilt gimbal -->
+        <visual name="tilt_realsense_visual">
+          <origin xyz="0.0 0 0.03" rpy="0 0 0"/>
+          <geometry>
+            <mesh filename="package://husky_panda_description/husky_panda_model/panda_mounted_husky/meshes/realsense.dae"/>
+          </geometry>
+        </visual>
+        <visual name="bot_camera_plate_low">
+          <origin xyz="0 0 0.017"/>
+          <geometry>
+            <box size="0.025 0.13 0.007"/>
+          </geometry>
+        </visual>
+        <visual name="bot_camera_plate_high">
+          <origin xyz="0 0 0.042"/>
+          <geometry>
+            <box size="0.025 0.13 0.007"/>
+          </geometry>
+        </visual>
+      </link>
+      <!-- camera_pan_tilt on the gimbal -->
+    <gazebo reference="tilt_gimbal_link">
+      <sensor name="camera_pan_tilt" type="rgbd_camera">
+        <topic>camera_pan_tilt</topic>
+        <pose>0 0 0.03 0 0 0</pose>
+        <update_rate>30</update_rate>
+        <camera name="camera_pan_tilt">
+          <horizontal_fov>1.5184</horizontal_fov>
+          <lens>
+            <intrinsics>
+              <fx>337.22195</fx>
+              <fy>337.22195</fy>
+              <cx>320.5</cx>
+              <cy>240.5</cy>
+              <s>0</s>
+            </intrinsics>
+          </lens>
+          <distortion>
+            <k1>0.0</k1><k2>0.0</k2><k3>0.0</k3>
+            <p1>0.0</p1><p2>0.0</p2>
+            <center>0.5 0.5</center>
+          </distortion>
+          <image>
+            <width>640</width>
+            <height>480</height>
+            <format>R8G8B8</format>
+          </image>
+          <clip><near>0.01</near><far>300</far></clip>
+          <depth_camera><clip><near>0.1</near><far>10</far></clip></depth_camera>
+          <noise>
+            <type>gaussian</type><mean>0</mean><stddev>0.007</stddev>
+          </noise>
+        </camera>
+      </sensor>
+    </gazebo>
+      <!-- planar_lidar_link -->
+      <link name="planar_lidar_link"/>
+            <!-- Camera Front -->
+      <link name="camera_front_link"/>
+      <joint name="camera_front_joint" type="fixed">
+        <parent link="base_link"/>
+        <child link="camera_front_link"/>
+        <origin xyz="0.468 0 0.360" rpy="0 0 0"/>
+      </joint>
+      <!-- Camera Down -->
+      <link name="camera_down_link"/>
+      <joint name="camera_down_joint" type="fixed">
+        <parent link="base_link"/>
+        <child link="camera_down_link"/>
+        <origin xyz="0.468 0 0.335" rpy="0 0.5236 0"/>
+      </joint>
+      <!-- Front 3D Lidar -->
+      <link name="front_laser_link"/>
+      <joint name="front_laser_joint" type="fixed">
+        <parent link="base_link"/>
+        <child link="front_laser_link"/>
+        <origin xyz="0.424 0 0.387" rpy="0 0 0"/>
+      </joint>
+      <!-- IMU -->
+      <link name="imu_link"/>
+      <joint name="imu_joint" type="fixed">
+        <parent link="base_link"/>
+        <child link="imu_link"/>
+        <origin xyz="0 0 0" rpy="0 0 0"/>
+      </joint>
+        <!-- planar_lidar_joint -->
+      <joint name="planar_lidar_joint" type="fixed">
+        <parent link="base_link"/>
+        <child link="planar_lidar_link"/>
+        <!-- <origin xyz="0.474 0 0.127" rpy="0 0 0"/> -->
+        <origin xyz="0.474 0 0.127" rpy="0 0 0"/>
+      </joint>
+      <!-- Example for front_left_wheel_link -->
+      <gazebo reference="front_left_wheel_link">
+        <mu1>2.0</mu1>
+        <mu2>2.0</mu2>
+        <surface>
+          <friction>
+            <ode>
+              <mu>2.0</mu>
+              <mu2>2.0</mu2>
+            </ode>
+          </friction>
+        </surface>
+      </gazebo>
+      <gazebo reference="front_right_wheel_link">
+        <mu1>2.0</mu1>
+        <mu2>2.0</mu2>
+        <surface>
+          <friction>
+            <ode>
+              <mu>2.0</mu>
+              <mu2>2.0</mu2>
+            </ode>
+          </friction>
+        </surface>
+      </gazebo>
+      <gazebo reference="rear_left_wheel_link">
+        <mu1>2.0</mu1>
+        <mu2>2.0</mu2>
+        <surface>
+          <friction>
+            <ode>
+              <mu>2.0</mu>
+              <mu2>2.0</mu2>
+            </ode>
+          </friction>
+        </surface>
+      </gazebo>
+      <gazebo reference="rear_right_wheel_link">
+        <mu1>2.0</mu1>
+        <mu2>2.0</mu2>
+        <surface>
+          <friction>
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
Commit message: updated moveit and added yolov8

File: husky_panda_description/husky_panda_model/panda_mounted_husky/panda_mounted_husky.urdf.xacro (robot description, xacro)
@@ -1,4 +1,5 @@
 <?xml version="1.0"?>
 <robot xmlns:xacro="http://www.ros.org/wiki/xacro" name="panda_mounted_husky">
+  <xacro:arg name="for_moveit" default="true"/>
     <!-- <xacro:property name="mesh_root"
          value="package://husky_panda_description/husky_panda_model/panda_mounted_husky/meshes"/>   -->
@@ -9,13 +10,23 @@
           LINKS
           ========================= -->
+      <link name="world_link"/>
+      <joint name="world_to_base" type="fixed">
+        <parent link="world_link"/>
+        <child link="base_link"/>
+      </joint>
       <!-- base_link -->
       <link name="base_link">
-        <inertial>
-          <origin xyz="-0.000543 -0.084945 0.062329" rpy="0 0 0"/>
-          <mass value="46.064"/>
-          <inertia
-            ixx="0.615397" ixy="-0.0240585" ixz="-0.120749"
-            iyy="1.75388"  iyz="-0.0028322" izz="2.03641"/>
-        </inertial>
+        <xacro:if value="$(arg for_moveit)">
+          <!-- no <inertial> when feeding MoveIt -->
+        </xacro:if>
+        <xacro:unless value="$(arg for_moveit)">
+          <inertial>
+            <origin xyz="-0.000543 -0.084945 0.062329" rpy="0 0 0"/>
+            <mass value="46.064"/>
+            <inertia
+              ixx="0.615397" ixy="-0.0240585" ixz="-0.120749"
+              iyy="1.75388"  iyz="-0.0028322" izz="2.03641"/>
+          </inertial>
+         </xacro:unless>
         <!-- <joint name="base_footprint_joint" type="fixed">
             <parent link="base_link"/>

Commit message: working moveit and updated readme

File: husky_panda_description/husky_panda_model/panda_mounted_husky/panda_mounted_husky.urdf.xacro (robot description, xacro)
@@ -10,9 +10,9 @@
           LINKS
           ========================= -->
-      <link name="world_link"/>
+      <!-- <link name="world_link"/>
       <joint name="world_to_base" type="fixed">
         <parent link="world_link"/>
         <child link="base_link"/>
-      </joint>
+      </joint> -->
       <!-- base_link -->
       <link name="base_link">
@@ -790,9 +790,9 @@
   </link>
   <joint name="panda_finger_joint1" type="prismatic">
-    <parent link="panda_link7"/><child link="panda_leftfinger"/>
+    <parent link="panda_link7"/>
+    <child  link="panda_leftfinger"/>
     <origin xyz="0 0 0.1654" rpy="0 0 -0.7853981633974483"/>
     <axis xyz="0 1 0"/>
-    <limit lower="-2.897246558310587" upper="2.897246558310587" effort="12" velocity="3.141592653589793"/>
-    <dynamics damping="3.0" friction="0.4"/>
+    <limit lower="0.0" upper="0.04" effort="20" velocity="0.2"/>
   </joint>
   <link name="panda_rightfinger">
@@ -806,9 +806,16 @@
   </link>
   <joint name="panda_finger_joint2" type="prismatic">
-    <parent link="panda_link7"/><child link="panda_rightfinger"/>
+    <parent link="panda_link7"/>
+    <child  link="panda_rightfinger"/>
     <origin xyz="0 0 0.1654" rpy="0 0 -0.7853981633974483"/>
     <axis xyz="0 -1 0"/>
     <limit lower="0.0" upper="0.04" effort="20" velocity="0.2"/>
-    <dynamics damping="3.0" friction="0.4"/>
+    <mimic joint="panda_finger_joint1" multiplier="1.0" offset="0.0"/>
+  </joint>
+  <link name="panda_hand_tcp"/>
+  <joint name="panda_hand_tcp_joint" type="fixed">
+    <parent link="gripper_mount"/>  <!-- or panda_link7 -->
+    <child  link="panda_hand_tcp"/>
+    <origin xyz="0 0 0.16" rpy="0 0 0"/>  <!-- tune to your gripper geometry -->
   </joint>
   <!-- =========================
